Commit message: launch files added

File: ros2_ws/src/my_rover_description/urdf/my_rover.urdf.xacro (robot description, xacro)
@@ -71,5 +71,5 @@
   <xacro:wheel name="right" x_pos="0" y_pos="${-wheel_separation/2}"/>
   <!-- ========== LIDAR LINK (RPLidar) ========== -->
-  <link name="lidar_link">
+  <link name="scan">
     <visual>
       <geometry>
@@ -93,5 +93,5 @@
   <joint name="lidar_joint" type="fixed">
     <parent link="base_link"/>
-    <child  link="lidar_link"/>
+    <child  link="scan"/>
     <!-- Mount on top-center of base -->
     <origin xyz="0 0 ${base_height/2 + 0.02}" rpy="0 0 0"/>
