Commit message: adding new launch files

File: ros2_ws/install/my_rover_description/share/my_rover_description/urdf/my_rover.urdf.xacro (robot description, xacro)
@@ -1 +1,106 @@
-/home/purujitk/203/MREN-203/ros2_ws/src/my_rover_description/urdf/my_rover.urdf.xacro
+<?xml version="1.0"?>
+<robot name="my_rover" xmlns:xacro="http://www.ros.org/wiki/xacro">
+  <!-- ========== PROPERTIES (edit these to match your robot) ========== -->
+  <xacro:property name="base_length" value="0.2775"/>   <!-- meters -->
+  <xacro:property name="base_width"  value="0.2"/>
+  <xacro:property name="base_height" value="0.05"/>
+  <xacro:property name="wheel_radius" value="0.0625"/>
+  <xacro:property name="wheel_width"  value="0.0635"/>
+  <xacro:property name="wheel_separation" value="0.0762"/> <!-- left to right -->
+  <!-- ========== BASE LINK ========== -->
+  <link name="base_link">
+    <visual>
+      <geometry>
+        <box size="${base_length} ${base_width} ${base_height}"/>
+      </geometry>
+      <material name="blue">
+        <color rgba="0.0 0.0 0.8 1.0"/>
+      </material>
+    </visual>
+    <collision>
+      <geometry>
+        <box size="${base_length} ${base_width} ${base_height}"/>
+      </geometry>
+    </collision>
+    <inertial>
+      <mass value="2.0"/>
+      <inertia ixx="0.01" ixy="0" ixz="0"
+               iyy="0.01" iyz="0" izz="0.02"/>
+    </inertial>
+  </link>
+  <!-- ========== WHEEL MACRO ========== -->
+  <xacro:macro name="wheel" params="name x_pos y_pos">
+    <link name="${name}_wheel_link">
+      <visual>
+        <geometry>
+          <cylinder radius="${wheel_radius}" length="${wheel_width}"/>
+        </geometry>
+        <material name="black">
+          <color rgba="0.1 0.1 0.1 1.0"/>
+        </material>
+      </visual>
+      <collision>
+        <geometry>
+          <cylinder radius="${wheel_radius}" length="${wheel_width}"/>
+        </geometry>
+      </collision>
+      <inertial>
+        <mass value="0.3"/>
+        <inertia ixx="0.001" ixy="0" ixz="0"
+                 iyy="0.001" iyz="0" izz="0.001"/>
+      </inertial>
+    </link>
+    <!-- Continuous joint = spinning wheel -->
+    <joint name="${name}_wheel_joint" type="continuous">
+      <parent link="base_link"/>
+      <child  link="${name}_wheel_link"/>
+      <origin xyz="${x_pos} ${y_pos} ${-base_height/2}"
+              rpy="${pi/2} 0 0"/>   <!-- rotate 90° so cylinder faces sideways -->
+      <axis xyz="0 0 1"/>
+    </joint>
+    <!-- Encoder frame (used by ros2_control / wheel odometry) -->
+    <link name="${name}_encoder_link"/>
+    <joint name="${name}_encoder_joint" type="fixed">
+      <parent link="${name}_wheel_link"/>
+      <child  link="${name}_encoder_link"/>
+      <origin xyz="0 0 0" rpy="0 0 0"/>
+    </joint>
+  </xacro:macro>
+  <!-- Instantiate left & right wheels -->
+  <xacro:wheel name="left"  x_pos="0" y_pos="${ wheel_separation/2}"/>
+  <xacro:wheel name="right" x_pos="0" y_pos="${-wheel_separation/2}"/>
+  <!-- ========== LIDAR LINK (RPLidar) ========== -->
+  <link name="scan">
+    <visual>
+      <geometry>
+        <cylinder radius="0.04" length="0.04"/>
+      </geometry>
+      <material name="red">
+        <color rgba="0.8 0.0 0.0 1.0"/>
+      </material>
+    </visual>
+    <collision>
+      <geometry>
+        <cylinder radius="0.04" length="0.04"/>
+      </geometry>
+    </collision>
+    <inertial>
+      <mass value="0.17"/>
+      <inertia ixx="0.0001" ixy="0" ixz="0"
+               iyy="0.0001" iyz="0" izz="0.0001"/>
+    </inertial>
+  </link>
+  <joint name="lidar_joint" type="fixed">
+    <parent link="base_link"/>
+    <child  link="scan"/>
+    <!-- Mount on top-center of base -->
+    <origin xyz="0 0 ${base_height/2 + 0.02}" rpy="0 0 0"/>
+  </joint>
+  <!-- ========== BASE_FOOTPRINT (required by Nav2) ========== -->
+  <link name="base_footprint"/>
+  <joint name="base_footprint_joint" type="fixed">
+    <parent link="base_footprint"/>
+    <child  link="base_link"/>
+    <origin xyz="0 0 ${wheel_radius}" rpy="0 0 0"/>
+  </joint>
+</robot>

File: ros2_ws/src/my_rover_description/urdf/my_rover.urdf.xacro (robot description, xacro)
@@ -2,10 +2,10 @@
 <robot name="my_rover" xmlns:xacro="http://www.ros.org/wiki/xacro">
   <!-- ========== PROPERTIES (edit these to match your robot) ========== -->
-  <xacro:property name="base_length" value="0.30"/>   <!-- meters -->
-  <xacro:property name="base_width"  value="0.25"/>
-  <xacro:property name="base_height" value="0.10"/>
-  <xacro:property name="wheel_radius" value="0.05"/>
-  <xacro:property name="wheel_width"  value="0.03"/>
-  <xacro:property name="wheel_separation" value="0.28"/> <!-- left to right -->
+  <xacro:property name="base_length" value="0.2775"/>   <!-- meters -->
+  <xacro:property name="base_width"  value="0.2"/>
+  <xacro:property name="base_height" value="0.05"/>
+  <xacro:property name="wheel_radius" value="0.0625"/>
+  <xacro:property name="wheel_width"  value="0.0635"/>
+  <xacro:property name="wheel_separation" value="0.0762"/> <!-- left to right -->
   <!-- ========== BASE LINK ========== -->
   <link name="base_link">
